Commit message: Funcionamiento general interfaz

File: src/robot_description/urdf/components/robot_structure/mobile_base.xacro (robot description, xacro)
@@ -87,5 +87,5 @@
     <!-- ================================================== -->
     <!-- Rueda delantera derecha -->
-    <joint name="base_front_right_wheel_joint" type="continuous">
+    <joint name="base_front_right_wheel_joint" type="fixed">
         <parent link="base_link"/>
         <child link="front_right_wheel_link"/>
@@ -93,16 +93,16 @@
         <origin xyz="${wheel_x_offset} ${-wheel_y_offset} 0" rpy="0 0 0"/>
         <!-- Eje de rotación: Y (ruedas giran alrededor del eje longitudinal) -->
-        <axis xyz="0 1 0"/>
+        <!--axis xyz="0 1 0"/-->
         <!-- Límites: velocity [rad/s], effort [Nm] -->
-        <limit velocity="100" effort="100"/>
+        <!--limit velocity="100" effort="100"/-->
     </joint>
     <!-- Rueda delantera izquierda -->
-    <joint name="base_front_left_wheel_joint" type="continuous">
+    <joint name="base_front_left_wheel_joint" type="fixed">
         <parent link="base_link"/>
         <child link="front_left_wheel_link"/>
         <!-- Posición: esquina delantera izquierda del chasis -->
         <origin xyz="${wheel_x_offset} ${wheel_y_offset} 0" rpy="0 0 0"/>
-        <axis xyz="0 1 0"/>
-        <limit velocity="100" effort="100"/>
+        <!--axis xyz="0 1 0"/>
+        <limit velocity="100" effort="100"/-->
     </joint>
     <!-- ================================================== -->
@@ -110,20 +110,20 @@
     <!-- ================================================== -->
     <!-- Rueda trasera derecha -->
-    <joint name="base_rear_right_wheel_joint" type="continuous">
+    <joint name="base_rear_right_wheel_joint" type="fixed">
         <parent link="base_link"/>
         <child link="rear_right_wheel_link"/>
         <!-- Posición: esquina trasera derecha del chasis -->
         <origin xyz="${-wheel_x_offset} ${-wheel_y_offset} 0" rpy="0 0 0"/>
-        <axis xyz="0 1 0"/>
-        <limit velocity="100" effort="100"/>
+        <!--axis xyz="0 1 0"/>
+        <limit velocity="100" effort="100"/-->
     </joint>
     <!-- Rueda trasera izquierda -->
-    <joint name="base_rear_left_wheel_joint" type="continuous">
+    <joint name="base_rear_left_wheel_joint" type="fixed">
         <parent link="base_link"/>
         <child link="rear_left_wheel_link"/>
         <!-- Posición: esquina trasera izquierda del chasis -->
         <origin xyz="${-wheel_x_offset} ${wheel_y_offset} 0" rpy="0 0 0"/>
-        <axis xyz="0 1 0"/>
-        <limit velocity="100" effort="100"/>
+        <!--axis xyz="0 1 0"/>
+        <limit velocity="100" effort="100"/-->
     </joint>
 </robot>

File: src/robot_description/urdf/my_robot.urdf.xacro (robot description, xacro)
@@ -10,7 +10,9 @@
     <!-- Incluir la cámara Asus Xtion -->
     <xacro:include filename="$(find robot_description)/urdf/components/camera/asus_xtion.urdf.xacro"/>
-  <!-- sensore -->
+    <!-- sensores -->
     <xacro:include filename="$(find robot_description)/urdf/components/imu/mpu6050.urdf.xacro"/>
     <xacro:include filename="$(find robot_description)/urdf/components/distance_sensor/sharp.urdf.xacro"/>
+    <!-- URDF RPLIDAR-->
+    <xacro:include filename="$(find robot_description)/urdf/components/rplidar/lidar.urdf.xacro"/>
     <!-- ================================================== -->
     <!-- ESTRUCTURA DEL ROBOT COMPLETO -->
@@ -28,16 +30,17 @@
     <!--
     Montar la cámara Asus Xtion en el base_link del robot diferencial
-    Ajusta las coordenadas xyz y rpy según donde quieras posicionar la cámara
+        xyz: posición relativa al base_link del robot
+            x: adelante/atrás (positivo = adelante)
+            y: izquierda/derecha (positivo = izquierda)
+            z: arriba/abajo (positivo = arriba)
+            rpy: orientación (roll, pitch, yaw en radianes)
     -->
     <xacro:sensor_asus_xtion parent="base_link" name="camera">
-        <!--
-        xyz: posición relativa al base_link del robot
-          x: adelante/atrás (positivo = adelante)
-          y: izquierda/derecha (positivo = izquierda)
-          z: arriba/abajo (positivo = arriba)
-        rpy: orientación (roll, pitch, yaw en radianes)
-        -->
         <origin xyz="0.4 0.0 0.35" rpy="0.0 0.0 0.0"/>
     </xacro:sensor_asus_xtion>
+    <!-- Unión entre base_link y el LIDAR RPLidar A1 / A1M8 -->
+    <xacro:sensor_rplidar parent="base_link" name="laser">
+        <origin xyz="0.10 0.0 0.58" rpy="0 0 0"/>
+    </xacro:sensor_rplidar>
      <!-- IMU (posición estable, cerca del centro de masa) -->
     <xacro:sensor_mpu6050 parent="base_link" name="imu">

Commit message: ya casi

File: src/robot_description/urdf/components/robot_structure/mobile_base.xacro (robot description, xacro)
@@ -5,13 +5,14 @@
     <!-- ================================================== -->
     <!-- Dimensiones del chasis principal [metros] -->
-    <xacro:property name="base_length" value="1"/>      <!-- Largo del chasis (100cm) -->
-    <xacro:property name="base_width" value="0.5"/>        <!-- Ancho del chasis (50cm) -->
-    <xacro:property name="base_height" value="0.3"/>       <!-- Altura del chasis (30cm) -->
+    <xacro:property name="base_length" value="0.7"/>      <!-- Largo del chasis (100cm) -->
+    <xacro:property name="base_width" value="0.651"/>        <!-- Ancho del chasis (50cm) -->
+    <xacro:property name="base_height" value="0.37"/>       <!-- Altura del chasis (30cm) -->
     <!-- Dimensiones de las ruedas [metros] -->
-    <xacro:property name="wheel_radius" value="0.10"/>      <!-- Radio de cada rueda (10cm) -->
-    <xacro:property name="wheel_length" value="0.05"/>     <!-- Grosor/ancho de rueda (5cm) -->
+    <xacro:property name="wheel_radius" value="0.165"/>      <!-- Radio de cada rueda (10cm) -->
+    <xacro:property name="wheel_length" value="0.09"/>     <!-- Grosor/ancho de rueda (5cm) -->
     <!-- Posicionamiento de ruedas [metros] -->
-    <xacro:property name="wheel_y_offset" value="${base_width / 2.0 + wheel_length / 2}"/>  <!-- Distancia desde centro a rueda (4.85cm) -->
-    <xacro:property name="wheel_x_offset" value="0.2"/> <!-- Desplazamiento longitudinal (20cm) -->
+    <xacro:property name="wheel_y_offset" value="${base_width / 2.0 + wheel_length / 2 + 0.04}"/>  <!-- Distancia desde centro a rueda (4.85cm) -->
+    <xacro:property name="wheel_x_offset" value="0.24"/> <!-- Desplazamiento longitudinal (20cm) -->
+    <xacro:property name="wheel_z_offset" value="0.05"/>
     <!-- ================================================== -->
     <!-- ESTRUCTURA PRINCIPAL DEL ROBOT -->
@@ -26,5 +27,5 @@
             </geometry>
             <!-- Posición: centro del chasis a la mitad de su altura -->
-            <origin xyz="0 0 ${base_height / 2.0}" rpy="0 0 0"/>
+            <origin xyz="0 0 ${base_height / 2.0 }" rpy="0 0 0"/>
             <material name="white"/>
         </visual>
@@ -81,5 +82,5 @@
         <child link="base_link"/>
         <!-- Posición: base_link elevado al radio de la rueda -->
-        <origin xyz="0 0 ${wheel_radius}" rpy="0 0 0"/>
+        <origin xyz="0 0 0.105" rpy="0 0 0"/>
     </joint>
     <!-- ================================================== -->
@@ -91,5 +92,5 @@
         <child link="front_right_wheel_link"/>
         <!-- Posición: esquina delantera derecha del chasis -->
-        <origin xyz="${wheel_x_offset} ${-wheel_y_offset} 0" rpy="0 0 0"/>
+        <origin xyz="${wheel_x_offset} ${-wheel_y_offset} ${wheel_z_offset}" rpy="0 0 0"/>
         <!-- Eje de rotación: Y (ruedas giran alrededor del eje longitudinal) -->
         <!--axis xyz="0 1 0"/-->
@@ -102,5 +103,5 @@
         <child link="front_left_wheel_link"/>
         <!-- Posición: esquina delantera izquierda del chasis -->
-        <origin xyz="${wheel_x_offset} ${wheel_y_offset} 0" rpy="0 0 0"/>
+        <origin xyz="${wheel_x_offset} ${wheel_y_offset} ${wheel_z_offset}" rpy="0 0 0"/>
         <!--axis xyz="0 1 0"/>
         <limit velocity="100" effort="100"/-->
@@ -114,5 +115,5 @@
         <child link="rear_right_wheel_link"/>
         <!-- Posición: esquina trasera derecha del chasis -->
-        <origin xyz="${-wheel_x_offset} ${-wheel_y_offset} 0" rpy="0 0 0"/>
+        <origin xyz="${-wheel_x_offset} ${-wheel_y_offset} ${wheel_z_offset}" rpy="0 0 0"/>
         <!--axis xyz="0 1 0"/>
         <limit velocity="100" effort="100"/-->
@@ -123,5 +124,5 @@
         <child link="rear_left_wheel_link"/>
         <!-- Posición: esquina trasera izquierda del chasis -->
-        <origin xyz="${-wheel_x_offset} ${wheel_y_offset} 0" rpy="0 0 0"/>
+        <origin xyz="${-wheel_x_offset} ${wheel_y_offset} ${wheel_z_offset}" rpy="0 0 0"/>
         <!--axis xyz="0 1 0"/>
         <limit velocity="100" effort="100"/-->

File: src/robot_description/urdf/my_robot.urdf.xacro (robot description, xacro)
@@ -39,17 +39,17 @@
     -->
     <xacro:sensor_asus_xtion parent="base_link" name="camera">
-        <origin xyz="0.4 0.0 0.35" rpy="0.0 0.0 0.0"/>
+        <origin xyz="0.31 0.0 0.22" rpy="0.0 0.0 0.0"/>
     </xacro:sensor_asus_xtion>
     <!--Union entre base_link y el GPS BU353N5-->
     <xacro:sensor_gps_bu353n5 parent="base_link" name="gnss">
-        <origin xyz="0.0 0.0 0.60" rpy="0 0 0"/>
+        <origin xyz="-0.32 0.0 0.60" rpy="0 0 0"/>
     </xacro:sensor_gps_bu353n5>
     <!-- Unión entre base_link y el LIDAR RPLidar A1 / A1M8 -->
     <xacro:sensor_rplidar parent="base_link" name="laser">
-        <origin xyz="0.10 0.0 0.58" rpy="0 0 0"/>
+        <origin xyz="-0.35 0.0 0.7" rpy="0 0 0"/>
     </xacro:sensor_rplidar>
      <!-- IMU (posición estable, cerca del centro de masa) -->
     <xacro:sensor_mpu6050 parent="base_link" name="imu">
-        <origin xyz="0.0 0.0 0.05" rpy="0.0 0.0 0.0"/>
+        <origin xyz="0.0 0.0245 0.18" rpy="0.0 0.0 0.0"/>
     </xacro:sensor_mpu6050>
     <!-- Sensores de distancia Sharp (múltiples posiciones) -->
