Commit message: integracion MPU9250

File: src/robot_description/urdf/my_robot.urdf.xacro (robot description, xacro)
@@ -15,4 +15,6 @@
     <!-- URDF RPLIDAR-->
     <xacro:include filename="$(find robot_description)/urdf/components/rplidar/lidar.urdf.xacro"/>
+    <!-- GPS BU-353N5 -->
+    <xacro:include filename="$(find robot_description)/urdf/components/gps/BU353N5.urdf.xacro"/>
     <!-- ================================================== -->
     <!-- ESTRUCTURA DEL ROBOT COMPLETO -->
@@ -39,4 +41,8 @@
         <origin xyz="0.4 0.0 0.35" rpy="0.0 0.0 0.0"/>
     </xacro:sensor_asus_xtion>
+    <!--Union entre base_link y el GPS BU353N5-->
+    <xacro:sensor_gps_bu353n5 parent="base_link" name="gnss">
+        <origin xyz="0.0 0.0 0.60" rpy="0 0 0"/>
+    </xacro:sensor_gps_bu353n5>
     <!-- Unión entre base_link y el LIDAR RPLidar A1 / A1M8 -->
     <xacro:sensor_rplidar parent="base_link" name="laser">

Commit message: funcional 1

File: src/robot_description/urdf/my_robot.urdf.xacro (robot description, xacro)
@@ -12,7 +12,4 @@
     <!-- sensores -->
     <xacro:include filename="$(find robot_description)/urdf/components/imu/mpu6050.urdf.xacro"/>
-    <xacro:include filename="$(find robot_description)/urdf/components/distance_sensor/sharp.urdf.xacro"/>
-    <!-- URDF RPLIDAR-->
-    <xacro:include filename="$(find robot_description)/urdf/components/rplidar/lidar.urdf.xacro"/>
     <!-- GPS BU-353N5 -->
     <xacro:include filename="$(find robot_description)/urdf/components/gps/BU353N5.urdf.xacro"/>
@@ -45,21 +42,7 @@
         <origin xyz="-0.32 0.0 0.60" rpy="0 0 0"/>
     </xacro:sensor_gps_bu353n5>
-    <!-- Unión entre base_link y el LIDAR RPLidar A1 / A1M8 -->
-    <xacro:sensor_rplidar parent="base_link" name="laser">
-        <origin xyz="-0.35 0.0 0.7" rpy="0 0 0"/>
-    </xacro:sensor_rplidar>
      <!-- IMU (posición estable, cerca del centro de masa) -->
     <xacro:sensor_mpu6050 parent="base_link" name="imu">
         <origin xyz="0.0 0.0245 0.18" rpy="0.0 0.0 0.0"/>
     </xacro:sensor_mpu6050>
-    <!-- Sensores de distancia Sharp (múltiples posiciones) -->
-    <xacro:sensor_sharp_gp2y0a21yk parent="base_link" name="sharp_front">
-        <origin xyz="0.5 0.0 0.04" rpy="0.0 0.0 0.0"/>
-    </xacro:sensor_sharp_gp2y0a21yk>
-    <xacro:sensor_sharp_gp2y0a21yk parent="base_link" name="sharp_left">
-        <origin xyz="0.0 0.25 0.04" rpy="0.0 0.0 ${pi/2}"/>
-    </xacro:sensor_sharp_gp2y0a21yk>
-    <xacro:sensor_sharp_gp2y0a21yk parent="base_link" name="sharp_right">
-        <origin xyz="0.0 -0.25 0.04" rpy="0.0 0.0 ${-pi/2}"/>
-    </xacro:sensor_sharp_gp2y0a21yk>
 </robot>
